File: pcb/atmega32u4.sch (KiCad schematic (older format))
At the start: 20 parts, among them CON1 ISP, P1 CONN_01X14, P2 CONN_01X14, P3 USB_OTG, U1 ATmega32U4-AU, Y1 16MHz

Commit message: Update footprints
Parts:
- D1, D2: footprint (none) -> LEDs:LED-5MM
- R4, R5: footprint (none) -> Resistors_SMD:R_0805_HandSoldering
Changed lines of the file:
@@
 ISP_SCK/PB1
 $Comp
-L GND #PWR07
+L GND #PWR06
 U 1 1 57DFE368
 P 4000 6100
-F 0 "#PWR07" H 4000 5850 50  0001 C CNN
+F 0 "#PWR06" H 4000 5850 50  0001 C CNN
 F 1 "GND" H 4000 5950 50  0000 C CNN
 F 2 "" H 4000 6100 50  0000 C CNN
@@
 XTAL1
 $Comp
-L GND #PWR08
+L GND #PWR07
 U 1 1 57DFEE60
 P 5300 6300
-F 0 "#PWR08" H 5300 6050 50  0001 C CNN
+F 0 "#PWR07" H 5300 6050 50  0001 C CNN
 F 1 "GND" H 5300 6150 50  0000 C CNN
 F 2 "" H 5300 6300 50  0000 C CNN
@@
 $EndComp
 $Comp
-L GND #PWR09
+L GND #PWR08
 U 1 1 57DFEE9B
 P 5800 6300
-F 0 "#PWR09" H 5800 6050 50  0001 C CNN
+F 0 "#PWR08" H 5800 6050 50  0001 C CNN
 F 1 "GND" H 5800 6150 50  0000 C CNN
 F 2 "" H 5800 6300 50  0000 C CNN
@@
 PF7
 $Comp
-L +5V #PWR010
+L +5V #PWR09
 U 1 1 57E26C1F
 P 3850 2600
-F 0 "#PWR010" H 3850 2450 50  0001 C CNN
+F 0 "#PWR09" H 3850 2450 50  0001 C CNN
 F 1 "+5V" H 3850 2740 50  0000 C CNN
 F 2 "" H 3850 2600 50  0000 C CNN
@@
 $EndComp
 $Comp
-L +5V #PWR?
+L +5V #PWR010
 U 1 1 57EB4CAF
 P 2250 3350
-F 0 "#PWR?" H 2250 3200 50  0001 C CNN
+F 0 "#PWR010" H 2250 3200 50  0001 C CNN
 F 1 "+5V" H 2250 3490 50  0000 C CNN
 F 2 "" H 2250 3350 50  0000 C CNN
@@
 $EndComp
 $Comp
-L +5V #PWR?
+L +5V #PWR011
 U 1 1 57EB53DC
 P 3850 1900
-F 0 "#PWR?" H 3850 1750 50  0001 C CNN
+F 0 "#PWR011" H 3850 1750 50  0001 C CNN
 F 1 "+5V" H 3850 2040 50  0000 C CNN
 F 2 "" H 3850 1900 50  0000 C CNN
@@
 $EndComp
 $Comp
-L VCC #PWR?
+L VCC #PWR012
 U 1 1 57EB59BD
 P 4000 5700
-F 0 "#PWR?" H 4000 5550 50  0001 C CNN
+F 0 "#PWR012" H 4000 5550 50  0001 C CNN
 F 1 "VCC" H 4000 5850 50  0000 C CNN
 F 2 "" H 4000 5700 50  0000 C CNN
@@
 $EndComp
 $Comp
-L VCC #PWR?
+L VCC #PWR013
 U 1 1 57EB5AB2
 P 3700 1600
-F 0 "#PWR?" H 3700 1450 50  0001 C CNN
+F 0 "#PWR013" H 3700 1450 50  0001 C CNN
 F 1 "VCC" H 3700 1750 50  0000 C CNN
 F 2 "" H 3700 1600 50  0000 C CNN
@@
 $EndComp
 $Comp
-L +5V #PWR?
+L +5V #PWR014
 U 1 1 57EB5C21
 P 8600 1850
-F 0 "#PWR?" H 8600 1700 50  0001 C CNN
+F 0 "#PWR014" H 8600 1700 50  0001 C CNN
 F 1 "+5V" H 8600 1990 50  0000 C CNN
 F 2 "" H 8600 1850 50  0000 C CNN
@@
 $EndComp
 $Comp
-L GND #PWR?
+L GND #PWR015
 U 1 1 57EB5F9C
 P 8250 3650
-F 0 "#PWR?" H 8250 3400 50  0001 C CNN
+F 0 "#PWR015" H 8250 3400 50  0001 C CNN
 F 1 "GND" H 8250 3500 50  0000 C CNN
 F 2 "" H 8250 3650 50  0000 C CNN
@@
 	7850 1950 8600 1950
 $Comp
-L GND #PWR?
+L GND #PWR016
 U 1 1 57EB672F
 P 7850 1950
-F 0 "#PWR?" H 7850 1700 50  0001 C CNN
+F 0 "#PWR016" H 7850 1700 50  0001 C CNN
 F 1 "GND" H 7850 1800 50  0000 C CNN
 F 2 "" H 7850 1950 50  0000 C CNN
@@
 $EndComp
 $Comp
-L VCC #PWR?
+L VCC #PWR017
 U 1 1 57EBA95D
 P 900 1100
-F 0 "#PWR?" H 900 950 50  0001 C CNN
+F 0 "#PWR017" H 900 950 50  0001 C CNN
 F 1 "VCC" H 900 1250 50  0000 C CNN
 F 2 "" H 900 1100 50  0000 C CNN
@@
 F 0 "R4" V 8680 5100 50  0000 C CNN
 F 1 "1K" V 8600 5100 50  0000 C CNN
-F 2 "" V 8530 5100 50  0000 C CNN
+F 2 "Resistors_SMD:R_0805_HandSoldering" V 8530 5100 50  0001 C CNN
 F 3 "" H 8600 5100 50  0000 C CNN
 	1    8600 5100
@@
 F 0 "D1" H 8600 5550 50  0000 C CNN
 F 1 "RED" H 8600 5350 50  0000 C CNN
-F 2 "" H 8600 5450 50  0000 C CNN
+F 2 "LEDs:LED-5MM" H 8600 5450 50  0001 C CNN
 F 3 "" H 8600 5450 50  0000 C CNN
 	1    8600 5450
@@
 $EndComp
 $Comp
-L GND #PWR?
+L GND #PWR018
 U 1 1 57EBBE20
 P 8600 5650
-F 0 "#PWR?" H 8600 5400 50  0001 C CNN
+F 0 "#PWR018" H 8600 5400 50  0001 C CNN
 F 1 "GND" H 8600 5500 50  0000 C CNN
 F 2 "" H 8600 5650 50  0000 C CNN
@@
 F 0 "R5" V 9530 5100 50  0000 C CNN
 F 1 "1K" V 9450 5100 50  0000 C CNN
-F 2 "" V 9380 5100 50  0000 C CNN
+F 2 "Resistors_SMD:R_0805_HandSoldering" V 9380 5100 50  0001 C CNN
 F 3 "" H 9450 5100 50  0000 C CNN
 	1    9450 5100
@@
 F 0 "D2" H 9450 5550 50  0000 C CNN
 F 1 "GREED" H 9450 5350 50  0000 C CNN
-F 2 "" H 9450 5450 50  0000 C CNN
+F 2 "LEDs:LED-5MM" H 9450 5450 50  0001 C CNN
 F 3 "" H 9450 5450 50  0000 C CNN
 	1    9450 5450
@@
 $EndComp
 $Comp
-L GND #PWR?
+L GND #PWR019
 U 1 1 57EBBF84
 P 9450 5650
-F 0 "#PWR?" H 9450 5400 50  0001 C CNN
+F 0 "#PWR019" H 9450 5400 50  0001 C CNN
 F 1 "GND" H 9450 5500 50  0000 C CNN
 F 2 "" H 9450 5650 50  0000 C CNN
@@
 $EndComp
 $Comp
-L +5V #PWR?
+L +5V #PWR020
 U 1 1 57EBBFA2
 P 9450 4950
-F 0 "#PWR?" H 9450 4800 50  0001 C CNN
+F 0 "#PWR020" H 9450 4800 50  0001 C CNN
 F 1 "+5V" H 9450 5090 50  0000 C CNN
 F 2 "" H 9450 4950 50  0000 C CNN

Commit message: About to do bottom layer
Parts:
- added SW1: SW_PUSH, Buttons_Switches_ThroughHole:SW_PUSH_SMALL, symbol SW_PUSH
- D1, D2: footprint LEDs:LED-5MM -> LEDs:LED-3MM
Connections:
- net PE2 is gone; now on net GND: U1.33 ((~HWB~)PE2)
- net GND: now also R3.2, SW1.2
- net ISP_RESET: now also SW1.1; no longer R3.2
Other:
- moved on the sheet: R3
Changed lines of the file:
@@
-$EndComp
-$Comp
-L GND #PWR02
-U 1 1 57DFDBDF
-P 2650 3000
-F 0 "#PWR02" H 2650 2750 50  0001 C CNN
-F 1 "GND" H 2650 2850 50  0000 C CNN
-F 2 "" H 2650 3000 50  0000 C CNN
-F 3 "" H 2650 3000 50  0000 C CNN
-	1    2650 3000
-	1    0    0    -1
 $EndComp
 $Comp
@@
 L R R3
 U 1 1 57DFE3A0
-P 3500 2250
-F 0 "R3" V 3420 2250 50  0000 C CNN
-F 1 "10kΩ" V 3500 2250 50  0000 C CNN
-F 2 "Resistors_SMD:R_0805_HandSoldering" V 3430 2250 50  0001 C CNN
-F 3 "" H 3500 2250 50  0000 C CNN
-	1    3500 2250
-	1    0    0    -1
-$EndComp
-Text Label 3550 3300 3    60   ~ 0
+P 7100 5150
+F 0 "R3" V 7020 5150 50  0000 C CNN
+F 1 "10kΩ" V 7100 5150 50  0000 C CNN
+F 2 "Resistors_SMD:R_0805_HandSoldering" V 7030 5150 50  0001 C CNN
+F 3 "" H 7100 5150 50  0000 C CNN
+	1    7100 5150
+	1    0    0    -1
+$EndComp
+Text Label 3500 3300 3    60   ~ 0
 ISP_RESET
 Text Label 3850 3900 2    60   ~ 0
@@
 	1    0    0    -1
 $EndComp
-Text Label 2900 3000 3    60   ~ 0
-GND
 Text Label 6300 1900 0    60   ~ 0
 PB0
@@
 PD7
 Text Label 6300 4000 0    60   ~ 0
-PE2
+HWB
 Text Label 6300 4100 0    60   ~ 0
 PE6
@@
 	1    0    0    -1
 $EndComp
-Wire Wire Line
-	3500 3300 3500 2400
-Wire Wire Line
-	3850 3300 3500 3300
-Connection ~ 1700 1550
-Wire Wire Line
-	2100 1550 2100 1500
-Wire Wire Line
-	1300 1550 1300 1500
-Wire Wire Line
-	900  1550 2100 1550
-Wire Wire Line
-	1700 1500 1700 1600
-Wire Wire Line
-	3850 4500 3850 4850
-Connection ~ 3850 4600
-Connection ~ 3850 4700
-Connection ~ 3850 4800
-Wire Wire Line
-	3850 2700 3100 2700
-Wire Wire Line
-	3100 2800 3850 2800
-Wire Wire Line
-	2800 2700 2400 2700
-Wire Wire Line
-	2400 2800 2800 2800
-Wire Wire Line
-	3850 3000 2550 3000
-Wire Wire Line
-	2550 3000 2550 2500
-Wire Wire Line
-	2550 2500 2400 2500
-Wire Wire Line
-	3850 2900 3250 2900
-Wire Wire Line
-	3250 2900 3250 3100
-Wire Wire Line
-	3900 5800 4000 5800
-Wire Wire Line
-	4000 5800 4000 5700
-Wire Wire Line
-	3900 6000 4000 6000
-Wire Wire Line
-	4000 6000 4000 6100
-Wire Wire Line
-	3900 5900 4100 5900
-Wire Wire Line
-	3400 5900 3150 5900
-Wire Wire Line
-	3400 5800 3300 5800
-Wire Wire Line
-	3400 6000 3300 6000
-Wire Wire Line
-	5700 5900 5800 5900
-Wire Wire Line
-	5800 5900 5800 6000
-Wire Wire Line
-	5400 5900 5300 5900
-Wire Wire Line
-	5300 5900 5300 6000
-Wire Wire Line
-	2400 2900 2400 3350
-Wire Wire Line
-	2400 3350 2250 3350
-Wire Wire Line
-	3850 2400 3700 2400
-Wire Wire Line
-	3700 2400 3700 1600
-Wire Wire Line
-	3850 2200 3700 2200
-Connection ~ 3700 2200
-Wire Wire Line
-	3850 2100 3700 2100
-Connection ~ 3700 2100
-Wire Wire Line
-	3850 2000 3700 2000
-Connection ~ 3700 2000
-Wire Wire Line
-	7850 1950 8600 1950
 $Comp
 L GND #PWR016
@@
 	1    0    0    -1
 $EndComp
-Wire Wire Line
-	900  1100 900  1200
-Wire Wire Line
-	900  1150 1300 1150
-Wire Wire Line
-	1300 1150 1300 1200
-Connection ~ 900  1150
-Wire Wire Line
-	1700 1100 1700 1200
-Wire Wire Line
-	1700 1150 2100 1150
-Wire Wire Line
-	2100 1150 2100 1200
-Connection ~ 1700 1150
-Wire Wire Line
-	900  1500 900  1550
-Connection ~ 1300 1550
-Wire Wire Line
-	3500 2100 3500 1900
-Wire Wire Line
-	3500 1900 3700 1900
-Connection ~ 3700 1900
-Wire Wire Line
-	8600 3650 8250 3650
 $Comp
 L R R4
@@
 F 0 "D1" H 8600 5550 50  0000 C CNN
 F 1 "RED" H 8600 5350 50  0000 C CNN
-F 2 "LEDs:LED-5MM" H 8600 5450 50  0001 C CNN
+F 2 "LEDs:LED-3MM" H 8600 5450 50  0001 C CNN
 F 3 "" H 8600 5450 50  0000 C CNN
 	1    8600 5450
@@
 F 0 "D2" H 9450 5550 50  0000 C CNN
 F 1 "GREED" H 9450 5350 50  0000 C CNN
-F 2 "LEDs:LED-5MM" H 9450 5450 50  0001 C CNN
+F 2 "LEDs:LED-3MM" H 9450 5450 50  0001 C CNN
 F 3 "" H 9450 5450 50  0000 C CNN
 	1    9450 5450
@@
 Text Label 8600 4950 2    60   ~ 0
 PE6
+Text Label 6650 5400 2    60   ~ 0
+HWB
+Wire Wire Line
+	3850 3300 3500 3300
+Connection ~ 1700 1550
+Wire Wire Line
+	2100 1550 2100 1500
+Wire Wire Line
+	1300 1550 1300 1500
+Wire Wire Line
+	900  1550 2100 1550
+Wire Wire Line
+	1700 1500 1700 1600
+Wire Wire Line
+	3850 4500 3850 4850
+Connection ~ 3850 4600
+Connection ~ 3850 4700
+Connection ~ 3850 4800
+Wire Wire Line
+	3850 2700 3100 2700
+Wire Wire Line
+	3100 2800 3850 2800
+Wire Wire Line
+	2800 2700 2400 2700
+Wire Wire Line
+	2400 2800 2800 2800
+Wire Wire Line
+	3850 3000 2550 3000
+Wire Wire Line
+	2550 3000 2550 2500
+Wire Wire Line
+	2550 2500 2400 2500
+Wire Wire Line
+	3850 2900 3250 2900
+Wire Wire Line
+	3250 2900 3250 3100
+Wire Wire Line
+	3900 5800 4000 5800
+Wire Wire Line
+	4000 5800 4000 5700
+Wire Wire Line
+	3900 6000 4000 6000
+Wire Wire Line
+	4000 6000 4000 6100
+Wire Wire Line
+	3900 5900 4100 5900
+Wire Wire Line
+	3400 5900 3150 5900
+Wire Wire Line
+	3400 5800 3300 5800
+Wire Wire Line
+	3400 6000 3300 6000
+Wire Wire Line
+	5700 5900 5800 5900
+Wire Wire Line
+	5800 5900 5800 6000
+Wire Wire Line
+	5400 5900 5300 5900
+Wire Wire Line
+	5300 5900 5300 6000
+Wire Wire Line
+	2400 2900 2400 3350
+Wire Wire Line
+	2400 3350 2250 3350
+Wire Wire Line
+	3850 2400 3700 2400
+Wire Wire Line
+	3700 2400 3700 1600
+Wire Wire Line
+	3850 2200 3700 2200
+Connection ~ 3700 2200
+Wire Wire Line
+	3850 2100 3700 2100
+Connection ~ 3700 2100
+Wire Wire Line
+	3850 2000 3700 2000
+Connection ~ 3700 2000
+Wire Wire Line
+	7850 1950 8600 1950
+Wire Wire Line
+	900  1100 900  1200
+Wire Wire Line
+	900  1150 1300 1150
+Wire Wire Line
+	1300 1150 1300 1200
+Connection ~ 900  1150
+Wire Wire Line
+	1700 1100 1700 1200
+Wire Wire Line
+	1700 1150 2100 1150
+Wire Wire Line
+	2100 1150 2100 1200
+Connection ~ 1700 1150
+Wire Wire Line
+	900  1500 900  1550
+Connection ~ 1300 1550
+Wire Wire Line
+	8600 3650 8250 3650
+Wire Wire Line
+	6650 5400 7100 5400
+Wire Wire Line
+	7100 5300 7100 5500
+Connection ~ 7100 5400
+$Comp
+L VCC #PWR021
+U 1 1 57EBD989
+P 7100 5000
+F 0 "#PWR021" H 7100 4850 50  0001 C CNN
+F 1 "VCC" H 7100 5150 50  0000 C CNN
+F 2 "" H 7100 5000 50  0000 C CNN
+F 3 "" H 7100 5000 50  0000 C CNN
+	1    7100 5000
+	1    0    0    -1
+$EndComp
+$Comp
+L GND #PWR022
+U 1 1 57EBD9C5
+P 7100 5500
+F 0 "#PWR022" H 7100 5250 50  0001 C CNN
+F 1 "GND" H 7100 5350 50  0000 C CNN
+F 2 "" H 7100 5500 50  0000 C CNN
+F 3 "" H 7100 5500 50  0000 C CNN
+	1    7100 5500
+	1    0    0    -1
+$EndComp
+Text Label 7150 1100 2    60   ~ 0
+ISP_RESET
+$Comp
+L SW_PUSH SW1
+U 1 1 57EBDCDC
+P 7450 1100
+F 0 "SW1" H 7600 1210 50  0000 C CNN
+F 1 "SW_PUSH" H 7450 1020 50  0000 C CNN
+F 2 "Buttons_Switches_ThroughHole:SW_PUSH_SMALL" H 7450 1100 50  0001 C CNN
+F 3 "" H 7450 1100 50  0000 C CNN
+	1    7450 1100
+	1    0    0    -1
+$EndComp
+$Comp
+L GND #PWR023
+U 1 1 57EBDD7D
+P 7750 1100
+F 0 "#PWR023" H 7750 850 50  0001 C CNN
+F 1 "GND" H 7750 950 50  0000 C CNN
+F 2 "" H 7750 1100 50  0000 C CNN
+F 3 "" H 7750 1100 50  0000 C CNN
+	1    7750 1100
+	1    0    0    -1
+$EndComp
+$Comp
+L GND #PWR?
+U 1 1 57EBECC4
+P 2550 3000
+F 0 "#PWR?" H 2550 2750 50  0001 C CNN
+F 1 "GND" H 2550 2850 50  0000 C CNN
+F 2 "" H 2550 3000 50  0000 C CNN
+F 3 "" H 2550 3000 50  0000 C CNN
+	1    2550 3000
+	1    0    0    -1
+$EndComp
 $EndSCHEMATC
