File: pcb/atmega32u4.kicad_pcb (KiCad board)
At the start: 2 copper layers, 38.1 x 69.9 mm, 15 parts, among them CON1 ISP, P1 CONN_01X14, P2 CONN_01X14, P3 USB_OTG, U1 ATmega32U4-AU, Y1 16MHz

Commit message: about to rewire pcb
Parts:
- added C0: 0.1uF, Capacitors_SMD:C_0805_HandSoldering, F.Cu at (144.1, 132.1)
- added D1: RED, LEDs:LED-5MM, F.Cu at (109.3, 131.3)
- added D2: GREED, LEDs:LED-5MM, F.Cu at (96.4, 136.1)
- added R4: 1K, Resistors_SMD:R_0805_HandSoldering, F.Cu at (113.3, 124.3)
- added R5: 1K, Resistors_SMD:R_0805_HandSoldering, F.Cu at (99.1, 143.5)
- C1, C2: value 100nF -> 0.1uF
- C3: value 4.7µF -> 10uF
- C5, C6: value 22pF -> 18pF
- moved P2 42.3 mm to (124.5, 125.7), turned to 180 degrees
- moved P1 27.9 mm to (152.4, 94.0)
- moved C2 3.42 mm to (135.3, 132.1), turned to 270 degrees
- moved CON1 3.17 mm to (135.9, 140.3)
- moved C1 2.29 mm to (141.6, 132.1), turned to 270 degrees
- moved C3 1.42 mm to (132.7, 132.1)
- moved R3 1.42 mm to (149.2, 132.1)
- turned U1 to 270 degrees
Connections:
- C1 pad 1: +5V -> VCC
- CON1 pad 2: +5V -> VCC
- P1 pad 1: /VCC -> +5V
- P1 pad 10: /PB7 -> /PC6
- P1 pad 11: /PC6 -> /PB7
- P1 pad 12: /PC7 -> /PB6
- P1 pad 13: /PF0 -> /PB5
- P1 pad 14: /PF1 -> /PB4
- P1 pad 3: /PB0 -> /PF0
- P1 pad 4: /ISP_SCK/PB1 -> /PF1
- P1 pad 5: /ISP_MOSI/PB2 -> /PF4
- P1 pad 6: /ISP_MISO/PB3 -> /PF5
- P1 pad 7: /PB4 -> /PF6
- P1 pad 8: /PB5 -> /PF7
- P1 pad 9: /PB6 -> /PC7
- P2 pad 10: /PD7 -> /ISP_MISO/PB3
- P2 pad 11: /PF4 -> /ISP_MOSI/PB2
- P2 pad 12: /PF5 -> /ISP_SCK/PB1
- P2 pad 13: /PF6 -> /PB0
- P2 pad 14: /PF7 -> /PE6
- P2 pad 2: GND -> /PD7
- P2 pad 3: /PD0 -> /PD6
- P2 pad 4: /PD1 -> /PD5
- P2 pad 5: /PD2 -> /PD4
- P2 pad 7: /PD4 -> /PD2
- P2 pad 8: /PD5 -> /PD1
- P2 pad 9: /PD6 -> /PD0
- P3 pad 1: /VCC -> +5V
- R3 pad 1: /VCC -> VCC
- U1 pad 14: /VCC -> VCC
- U1 pad 2: /VCC -> +5V
- U1 pad 24: /VCC -> VCC
- U1 pad 34: /VCC -> VCC
- U1 pad 44: /VCC -> VCC
- U1 pad 7: /VCC -> +5V
Routing:
- net GND: track 164.0 -> 2.54 mm, vias 10 -> 0
- net /VCC: track 160.0 -> 0.00 mm, vias 9 -> 0
- net /PF1: track 58.6 -> 0.00 mm, vias 2 -> 0
- net /ISP_SCK/PB1: track 58.3 -> 0.00 mm, vias 2 -> 0
- net /ISP_RESET: track 56.4 -> 0.00 mm, vias 2 -> 0
- net /PF0: track 53.2 -> 0.00 mm, vias 2 -> 0
- net /ISP_MOSI/PB2: track 48.4 -> 0.00 mm, vias 2 -> 0
- net /ISP_MISO/PB3: track 45.9 -> 0.00 mm, vias 2 -> 0
- net /PF7: track 44.4 -> 0.00 mm, vias 2 -> 0
- net /PF6: track 40.6 -> 0.00 mm, vias 2 -> 0
- net /PD0: track 33.7 -> 0.00 mm, vias 2 -> 0
- net /PC7: track 33.6 -> 0.00 mm, vias 4 -> 0
- net /PF5: track 33.4 -> 0.00 mm, vias 2 -> 0
- net /PF4: track 31.6 -> 0.00 mm, vias 2 -> 0
- net /PC6: track 30.9 -> 0.00 mm, vias 4 -> 0
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Other:
- board outline removed

Commit message: About to do bottom layer
Parts:
- added SW1: SW_PUSH, Buttons_Switches_ThroughHole:SW_PUSH_SMALL, F.Cu at (139.7, 118.7)
- D1, D2: footprint LEDs:LED-5MM -> LEDs:LED-3MM
- moved C0 19.1 mm to (145.4, 113.0)
- moved R3 11.1 mm to (144.8, 142.2)
- moved C1 10.2 mm to (141.6, 142.2)
- moved C2 10.2 mm to (135.3, 142.2)
- moved C3 10.2 mm to (132.7, 142.2)
- moved CON1 10.2 mm to (135.9, 150.5)
- moved D1 9.28 mm to (118.1, 128.3), turned to 180 degrees
- moved Y1 8.26 mm to (138.4, 126.9)
- moved C5 7.62 mm to (141.0, 133.3)
- moved C6 7.62 mm to (135.9, 133.3)
- moved P1 4.02 mm to (148.6, 92.7)
- moved P2 3.81 mm to (128.3, 125.7)
- moved P3 3.17 mm to (138.4, 85.7)
- moved R4 1.82 mm to (113.7, 122.6), turned to 270 degrees
- moved C4 0.64 mm to (133.3, 92.1)
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Connections:
- R3 pad 2: /ISP_RESET -> GND
- U1 pad 33: /PE2 -> GND
Routing:
- net VCC: track 0.00 -> 35.0 mm
- net GND: track 2.54 -> 31.3 mm, vias 0 -> 1
- net +5V: track 0.00 -> 24.7 mm
- net /PB4: track 0.00 -> 19.7 mm
- net /PB5: track 0.00 -> 16.9 mm
- net /PD7: track 0.00 -> 15.8 mm
- net /PB6: track 0.00 -> 15.1 mm
- net /PC6: track 0.00 -> 14.4 mm
- net /PD6: track 0.00 -> 13.3 mm
- net Net-(P3-Pad6): track 0.00 -> 13.2 mm
- net /PB0: track 0.00 -> 10.8 mm
- net /PD5: track 0.00 -> 10.6 mm, vias 0 -> 1
- net /PD4: track 0.00 -> 10.5 mm
- net Net-(C4-Pad1): track 0.00 -> 9.39 mm
- net /PF0: track 0.00 -> 9.36 mm
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
Commit message: WIP
Parts:
- D2: value GREED -> GREEN
- moved D2 50.3 mm to (146.7, 134.6), turned to 90 degrees
- moved R5 48.8 mm to (145.4, 128.3), turned to 270 degrees
- moved R4 18.7 mm to (131.4, 128.3)
- moved D1 13.6 mm to (130.2, 134.6), turned to 90 degrees
- moved R3 3.24 mm to (144.1, 139.1)
- moved C1 3.18 mm to (141.6, 139.1)
- moved C2 3.18 mm to (135.3, 139.1)
- moved C3 3.18 mm to (132.7, 139.1)
- moved CON1 3.18 mm to (135.9, 147.3)
Routing:
- net /ISP_RESET: track 2.10 -> 55.9 mm
- net /ISP_SCK/PB1: track 9.03 -> 59.3 mm, vias 0 -> 1
- net /ISP_MISO/PB3: track 7.55 -> 57.5 mm, vias 0 -> 1
- net /ISP_MOSI/PB2: track 8.82 -> 55.4 mm, vias 0 -> 1
- net GND: track 31.3 -> 48.7 mm, vias 1 -> 4
- net +5V: track 24.7 -> 26.4 mm, vias 0 -> 1
